Commit message: Add urdf base_scan

File: src/kuzya_bot/description/urdf/diffbot_description.urdf.xacro (robot description, xacro)
@@ -133,4 +133,29 @@
         </inertial>
       </link>
+<!-- LIDAR Link -->
+  <link name="${prefix}base_scan">
+    <visual>
+      <geometry>
+        <cylinder radius="0.035" length="0.030"/>
+      </geometry>
+      <origin xyz="0 0 0" rpy="0 0 0"/>
+      <material name="black"/>
+    </visual>
+    <collision>
+      <geometry>
+        <cylinder radius="0.035" length="0.030"/>
+      </geometry>
+      <origin xyz="0 0 0" rpy="0 0 0"/>
+    </collision>
+    <inertial>
+      <mass value="0.125"/>
+      <inertia ixx="0.001" ixy="0" ixz="0" iyy="0.001" iyz="0" izz="0.001"/>
+    </inertial>
+  </link>
+  <joint name="${prefix}lidar_joint" type="fixed">
+    <parent link="base_link"/>
+    <child link="base_scan"/>
+    <origin xyz="0 0 0.15" rpy="0 0 0"/>
+  </joint>
   </xacro:macro>
 </robot>

Commit message: good map

File: src/kuzya_bot/description/urdf/diffbot_description.urdf.xacro (robot description, xacro)
@@ -134,5 +134,5 @@
       </link>
 <!-- LIDAR Link -->
-  <link name="${prefix}base_scan">
+  <link name="${prefix}base_laser">
     <visual>
       <geometry>
@@ -155,5 +155,5 @@
   <joint name="${prefix}lidar_joint" type="fixed">
     <parent link="base_link"/>
-    <child link="base_scan"/>
+    <child link="base_laser"/>
     <origin xyz="0 0 0.15" rpy="0 0 0"/>
   </joint>
